File: napajeniMOB/napajeniMOB.brd (EAGLE design)
At the start: 103.8 x 51.3 mm, 45 parts, among them IC1 MC34063AD, T1 BD244

Commit message: Doplneny hodnosty soucastek
Parts:
- C2: value (none) -> 100u
- C3: value (none) -> 47u
- R3: value 150 -> 330
- R9: value 150 -> 1k2
Changed lines of the file:
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@@
 <element name="CHARGE" library="#Svorkovnice" package="AK500/2" value="" x="57.15" y="7.62" rot="R180"/>
 <element name="D1" library="led" package="LED3MM" value="" x="50.8" y="22.86"/>
-<element name="R3" library="#PaJa_30" package="0805" value="150" x="55.245" y="21.59" rot="MR0"/>
+<element name="R3" library="#PaJa_30" package="0805" value="330" x="55.245" y="21.59" rot="MR0"/>
 <element name="X2" library="D-USBcon" package="USBGROUNDED" value="" x="93.98" y="39.37" rot="R180"/>
 <element name="X3" library="D-USBcon" package="USBGROUNDED" value="" x="76.2" y="39.37" rot="R180"/>
@@
 <element name="R8" library="rcl" package="M0805" value="3k" x="31.75" y="24.13" rot="MR0"/>
 <element name="C1" library="rcl" package="C0805" value="860p" x="25.4" y="33.02" rot="MR0"/>
-<element name="C2" library="rcl" package="E5-8,5" value="" x="44.45" y="29.21" rot="R180"/>
+<element name="C2" library="rcl" package="E5-8,5" value="100u" x="44.45" y="29.21" rot="R180"/>
 <element name="T1" library="transistor" package="TO220" value="BD244" x="8.89" y="27.94" rot="R90"/>
 <element name="L1" library="rcl" package="TJ3-U1" value="47u" x="34.29" y="30.48"/>
 <element name="D3" library="led" package="LED3MM" value="" x="60.96" y="14.605" rot="R90"/>
-<element name="R9" library="#PaJa_30" package="0805" value="150" x="59.69" y="18.415" rot="MR180"/>
-<element name="C3" library="rcl" package="E5-8,5" value="" x="53.34" y="16.51"/>
+<element name="R9" library="#PaJa_30" package="0805" value="1k2" x="59.69" y="18.415" rot="MR180"/>
+<element name="C3" library="rcl" package="E5-8,5" value="47u" x="53.34" y="16.51"/>
 <element name="C4" library="rcl" package="C0805" value="100n" x="26.67" y="19.05" rot="MR0"/>
 </elements>
