File: napajeniMOB/napajeniMOB.brd (EAGLE design)
At the start: 103.8 x 51.3 mm, 45 parts, among them IC1 MC34063AD, T1 BD244

Commit message: Update napajeniMOB.brd
Takto byla deska vyrobena 20.12.2013
Parts:
- R6: value 100R -> 100
- R7: value 56R -> 56
- moved 5V_SUP_SW 5.75 mm to (45.1, 15.2)
- moved R3 5.24 mm to (50.2, 20.3)
- moved D1 4.02 mm to (47.0, 21.6), turned to 270 degrees
- moved R9 1.42 mm to (61.0, 19.1), turned to 270 degrees
- moved C4 1.27 mm to (25.4, 19.1)
Routing:
- net GND: track 438.0 -> 402.6 mm
- net +12V: track 113.4 -> 110.9 mm
- net N$7: track 4.28 -> 2.22 mm
- net +5V: track 47.0 -> 45.2 mm
- net N$6: track 34.9 -> 36.5 mm
- net N$8: track 2.75 -> 2.22 mm
Other:
- board size 103.8 x 51.3 mm -> 106 x 53.3 mm
