File: napajeniMOB/napajeniMOB.brd (EAGLE design)
At the start: 106 x 53.3 mm, 45 parts, among them IC1 MC34063AD, T1 BD244

Commit message: Merge with DavidOb version
Parts:
- C2: value 100u -> (none)
Changed lines of the file:
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@@
 <element name="R8" library="rcl" package="M0805" value="3k" x="31.75" y="24.13" rot="MR0"/>
 <element name="C1" library="rcl" package="C0805" value="860p" x="25.4" y="33.02" rot="MR0"/>
-<element name="C2" library="rcl" package="E5-8,5" value="100u" x="44.45" y="29.21" rot="R180"/>
+<element name="C2" library="rcl" package="E5-8,5" value="" x="44.45" y="29.21" rot="R180"/>
 <element name="T1" library="transistor" package="TO220" value="BD244" x="8.89" y="27.94" rot="R90"/>
 <element name="L1" library="rcl" package="TJ3-U1" value="47u" x="34.29" y="30.48"/>
