File: 12V-to-USB/converter.brd (EAGLE design)
At the start: 23.8 x 18.4 mm, 14 parts, among them IC1 MC34063AD

Commit message: + Added values of parts.
Parts:
- C1: value (none) -> 220p
- C2: value (none) -> 100n
- C3: value (none) -> 100u
- C4, L1: value (none) -> 47u
- D1: value (none) -> SK210
- LSP1: value LSP11 -> +12V
- LSP2: value LSP11 -> GND
- R1: value (none) -> 3k
- R2: value (none) -> 1k
- R3: value (none) -> 0R1
Changed lines of the file:
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@@
 <elements>
 <element name="IC1" library="mc34063" package="SOIC8" value="MC34063AD" x="36.195" y="27.305" rot="MR270"/>
-<element name="C1" library="rcl" package="C0805" value="" x="38.1" y="23.495" rot="MR0"/>
-<element name="R1" library="rcl" package="R0805" value="" x="27.305" y="29.21" rot="MR180"/>
-<element name="R2" library="rcl" package="R0805" value="" x="22.86" y="29.21" rot="MR180"/>
-<element name="R3" library="rcl" package="R0805" value="" x="31.115" y="27.94" rot="MR90"/>
-<element name="C2" library="rcl" package="C0805" value="" x="32.385" y="22.86" rot="MR270"/>
-<element name="C3" library="rcl" package="PANASONIC_D" value="" x="26.67" y="34.29" rot="MR270"/>
-<element name="C4" library="rcl" package="PANASONIC_D" value="" x="26.67" y="24.13" rot="MR180"/>
-<element name="L1" library="rcl" package="PIS2816" value="" x="34.29" y="34.29" rot="MR0"/>
-<element name="D1" library="diode" package="SMB" value="" x="40.64" y="34.925" rot="MR270"/>
-<element name="LSP1" library="solpad" package="LSP11" value="LSP11" x="21.59" y="26.035"/>
-<element name="LSP2" library="solpad" package="LSP11" value="LSP11" x="21.59" y="21.59"/>
+<element name="C1" library="rcl" package="C0805" value="220p" x="38.1" y="23.495" rot="MR0"/>
+<element name="R1" library="rcl" package="R0805" value="3k" x="27.305" y="29.21" rot="MR180"/>
+<element name="R2" library="rcl" package="R0805" value="1k" x="22.86" y="29.21" rot="MR180"/>
+<element name="R3" library="rcl" package="R0805" value="0R1" x="31.115" y="27.94" rot="MR90"/>
+<element name="C2" library="rcl" package="C0805" value="100n" x="32.385" y="22.86" rot="MR270"/>
+<element name="C3" library="rcl" package="PANASONIC_D" value="100u" x="26.67" y="34.29" rot="MR270"/>
+<element name="C4" library="rcl" package="PANASONIC_D" value="47u" x="26.67" y="24.13" rot="MR180"/>
+<element name="L1" library="rcl" package="PIS2816" value="47u " x="34.29" y="34.29" rot="MR0"/>
+<element name="D1" library="diode" package="SMB" value="SK210" x="40.64" y="34.925" rot="MR270"/>
+<element name="LSP1" library="solpad" package="LSP11" value="+12V" x="21.59" y="26.035"/>
+<element name="LSP2" library="solpad" package="LSP11" value="GND" x="21.59" y="21.59"/>
 <element name="LSP3" library="solpad" package="LSP11" value="LSP11" x="21.59" y="32.385"/>
 <element name="LSP4" library="solpad" package="LSP11" value="LSP11" x="21.59" y="36.83"/>

Commit message: Changed layout and some parts.
Parts:
- L1: device rcl:PIS2816 -> inductors:DR127
- moved D1 8.90 mm to (40.3, 26.0)
- moved R1 4.55 mm to (22.9, 30.2), turned to 0 degrees
- moved R3 3.27 mm to (28.3, 29.5)
- moved L1 3.00 mm to (35.9, 36.8)
- moved C1 2.56 mm to (35.6, 23.8)
- moved IC1 2.56 mm to (33.7, 27.6)
- moved R2 0.95 mm to (22.9, 28.3)
- moved C3 0.71 mm to (26.0, 34.6)
- moved C2 0.45 mm to (32.1, 23.2)
Routing:
- net GND: track 63.6 -> 47.3 mm
- net N$6: track 18.9 -> 12.9 mm
- net N$1: track 13.1 -> 10.2 mm
- net +12V: track 21.4 -> 24.2 mm
- net +5V: track 16.5 -> 13.7 mm
- net N$2: track 9.08 -> 9.66 mm
Other:
- board size 23.8 x 18.4 mm -> 23.8 x 23.2 mm
